File: corne-light/pcb/corne-light.kicad_pcb (KiCad board)
At the start: 2 copper layers, 275.5 x 105.6 mm, 86 parts, among them J1 MJ-4PP-9, J2 OLED, J6 MJ-4PP-9, J7 OLED, SW10 SW_PUSH, SW11 SW_PUSH, SW12 SW_PUSH, SW14 SW_PUSH, SW15 SW_PUSH, SW16 SW_PUSH, SW17 SW_PUSH, SW18 SW_PUSH, SW19 SW_PUSH, SW2 SW_PUSH, SW20 SW_PUSH, SW21 SW_PUSH, SW23 SW_PUSH, SW24 SW_PUSH, SW25 SW_PUSH, SW26 SW_PUSH, SW27 SW_PUSH, SW29 SW_PUSH, SW3 SW_PUSH, SW30 SW_PUSH, SW31 SW_PUSH, SW32 SW_PUSH, SW33 SW_PUSH, SW35 SW_PUSH, SW36 SW_PUSH, SW37 SW_PUSH, SW38 SW_PUSH, SW39 SW_PUSH, SW4 SW_PUSH, SW40 SW_PUSH, SW41 SW_PUSH, SW42 SW_PUSH, SW5 SW_PUSH, SW6 SW_PUSH, SW8 SW_PUSH, SW9 SW_PUSH, U1 ProMicro, U2 ProMicro

Commit message: Added track pad support with reset board soldered on the pcb
Parts:
- removed REF** (x6): Breakaway_Tabs, kbd:Breakaway_Tabs
- added ?: , , F.Cu at (171.3, 77.3)
- added ?: , , F.Cu at (171.3, 80.9)
- added C1: 2.2uF, Capacitor_SMD:C_1206_3216Metric, F.Cu at (164.7, 58.7)
- added R3: 4.7K, Resistor_SMD:R_0805_2012Metric, F.Cu at (162.0, 63.3)
- added R4: 4.7K, Resistor_SMD:R_0805_2012Metric, F.Cu at (167.2, 63.4)
- added R5: 4.7K, Resistor_SMD:R_0805_2012Metric, F.Cu at (171.3, 79.1)
- added TP: J8, Connector_PinHeader_2.54mm:PinHeader_1x05_P2.54mm_Vertical, F.Cu at (171.7, 74.0)
- U1, U2: value ProMicro -> Elite-C; footprint kbd:ProMicro_v3 -> keebio-parts:Elite-C; moved to B.Cu
- turned RSW2 to 90 degrees
- turned U1 to -90 degrees
- turned U2 to -90 degrees
Connections:
- U1 pad 1: unconnected-(U1-Pad1) -> data
- U1 pad 2: data -> unconnected-(U1-Pad2)
- U2 pad 1: unconnected-(U2-Pad1) -> data_r
- U2 pad 2: data_r -> tp_data_r
Routing:
- net row3: track 99.2 -> 178.6 mm, vias 2 -> 0
- net col1_r: track 190.8 -> 251.8 mm
- net col2_r: track 182.6 -> 226.9 mm
- net row2: track 138.6 -> 178.2 mm, vias 2 -> 0
- net col3_r: track 207.1 -> 246.3 mm
- net tp_data_r: track 0.00 -> 36.2 mm
- net col4_r: track 184.1 -> 219.3 mm
- net col5_r: track 175.6 -> 209.8 mm
- net row0: track 171.1 -> 138.4 mm, vias 2 -> 0
- net data: track 78.3 -> 46.6 mm
- net VDD: track 44.8 -> 75.6 mm
- net /tp_rst: track 0.00 -> 19.9 mm
- net data_r: track 48.2 -> 63.5 mm
- net SDA_r: track 33.3 -> 47.5 mm, vias 0 -> 1
- net SCL_r: track 28.8 -> 41.7 mm, vias 0 -> 1
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