File: corne-light/pcb/corne-light.kicad_sch (KiCad schematic)
At the start: 80 parts, among them J1 MJ-4PP-9, J2 OLED, J6 MJ-4PP-9, J7 OLED, SW10 SW_PUSH, SW11 SW_PUSH, SW12 SW_PUSH, SW14 SW_PUSH, SW15 SW_PUSH, SW16 SW_PUSH, SW17 SW_PUSH, SW18 SW_PUSH, SW19 SW_PUSH, SW2 SW_PUSH, SW20 SW_PUSH, SW21 SW_PUSH, SW23 SW_PUSH, SW24 SW_PUSH, SW25 SW_PUSH, SW26 SW_PUSH, SW27 SW_PUSH, SW29 SW_PUSH, SW3 SW_PUSH, SW30 SW_PUSH, SW31 SW_PUSH, SW32 SW_PUSH, SW33 SW_PUSH, SW35 SW_PUSH, SW36 SW_PUSH, SW37 SW_PUSH, SW38 SW_PUSH, SW39 SW_PUSH, SW4 SW_PUSH, SW40 SW_PUSH, SW41 SW_PUSH, SW42 SW_PUSH, SW5 SW_PUSH, SW6 SW_PUSH, SW8 SW_PUSH, SW9 SW_PUSH, U1 ProMicro, U2 ProMicro

Commit message: Added track pad support with reset board soldered on the pcb
Parts:
- added C1: 2.2uF, Capacitor_SMD:C_1206_3216Metric, symbol Device:C_Polarized
- added R3, R4, R5: 4.7K, Resistor_SMD:R_0805_2012Metric, symbol Device:R
- added TrackPoint1: J8, Connector_PinHeader_2.54mm:PinHeader_1x05_P2.54mm_Vertical, symbol Connector_Generic:Conn_01x05
- U1, U2: value ProMicro -> Elite-C; footprint kbd:ProMicro_v3 -> keebio-parts:Elite-C; symbol kbd:ProMicro -> keebio:Elite-C
Connections:
- net GNDA: now also R5.1, TrackPoint1.4 (Pin_4)
- net VDD: now also C1.1, R3.2, R4.2, TrackPoint1.5 (Pin_5)
- net data: now also U1.1 (TX0/PD3); no longer U1.2 (RX1/D2)
- net data_r: now also U2.1 (TX0/PD3); no longer U2.2 (RX1/D2)
- new net tp_clk_r: R3.1, TrackPoint1.3 (Pin_3), U2.26 (D5)
- new net tp_data_r: R4.1, TrackPoint1.1 (Pin_1), U2.2 (RX1/PD2)
- new net tp_rst: C1.2, R5.2, TrackPoint1.2 (Pin_2)
- no-connect marks 17 -> 25
Other:
- moved on the sheet: J7
